Commit message: Modified coordinates of base_link.

File: urdf/rohand_left.urdf (robot description, URDF)
Before this commit: robot rohand_left, 26 links, 25 joints
Links:
- link base_link: mass 0.05182218018482 -> 0.0518221802910333; geometry collision mesh filename=package://rohand_urdf_ros2/meshes_l//base_link.STL; visual mesh filename=package://rohand_urdf_ros2/meshes_l//base_link.STL
- link if_connecting_link: geometry collision mesh filename=package://rohand_urdf_ros2/meshes_l//if_connecting_link.STL; visual mesh filename=package://rohand_urdf_ros2/meshes_l//if_connecting_link.STL
- link if_distal_link: mass 0.00416343809021936 -> 0.00416343809392657; geometry collision mesh filename=package://rohand_urdf_ros2/meshes_l//if_distal_link.STL; visual mesh filename=package://rohand_urdf_ros2/meshes_l//if_distal_link.STL
- link if_proximal_link: geometry collision mesh filename=package://rohand_urdf_ros2/meshes_l//if_proximal_link.STL; visual mesh filename=package://rohand_urdf_ros2/meshes_l//if_proximal_link.STL
- link if_slider_abpart_link: geometry collision mesh filename=package://rohand_urdf_ros2/meshes_l//if_slider_abpart_link.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; visual mesh filename=package://rohand_urdf_ros2/meshes_l//if_slider_abpart_link.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
- link if_slider_link: geometry collision mesh filename=package://rohand_urdf_ros2/meshes_l//if_slider_link.STL; visual mesh filename=package://rohand_urdf_ros2/meshes_l//if_slider_link.STL
- link lf_connecting_link: geometry collision mesh filename=package://rohand_urdf_ros2/meshes_l//lf_connecting_link.STL; visual mesh filename=package://rohand_urdf_ros2/meshes_l//lf_connecting_link.STL
- link lf_distal_link: geometry collision mesh filename=package://rohand_urdf_ros2/meshes_l//lf_distal_link.STL; visual mesh filename=package://rohand_urdf_ros2/meshes_l//lf_distal_link.STL
- link lf_proximal_link: geometry collision mesh filename=package://rohand_urdf_ros2/meshes_l//lf_proximal_link.STL; visual mesh filename=package://rohand_urdf_ros2/meshes_l//lf_proximal_link.STL
- link lf_slider_abpart_link: geometry collision mesh filename=package://rohand_urdf_ros2/meshes_l//lf_slider_abpart_link.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; visual mesh filename=package://rohand_urdf_ros2/meshes_l//lf_slider_abpart_link.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
- link lf_slider_link: geometry collision mesh filename=package://rohand_urdf_ros2/meshes_l//lf_slider_link.STL; visual mesh filename=package://rohand_urdf_ros2/meshes_l//lf_slider_link.STL
- link mf_connecting_link: geometry collision mesh filename=package://rohand_urdf_ros2/meshes_l//mf_connecting_link.STL; visual mesh filename=package://rohand_urdf_ros2/meshes_l//mf_connecting_link.STL
- link mf_distal_link: mass 0.00416341391410531 -> 0.0041634139178577; geometry collision mesh filename=package://rohand_urdf_ros2/meshes_l//mf_distal_link.STL; visual mesh filename=package://rohand_urdf_ros2/meshes_l//mf_distal_link.STL
- link mf_proximal_link: mass 0.102110343400807 -> 0.102110343610594; geometry collision mesh filename=package://rohand_urdf_ros2/meshes_l//mf_proximal_link.STL; visual mesh filename=package://rohand_urdf_ros2/meshes_l//mf_proximal_link.STL
- link mf_slider_abpart_link: geometry collision mesh filename=package://rohand_urdf_ros2/meshes_l//mf_slider_abpart_link.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; visual mesh filename=package://rohand_urdf_ros2/meshes_l//mf_slider_abpart_link.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
- link mf_slider_link: geometry collision mesh filename=package://rohand_urdf_ros2/meshes_l//mf_slider_link.STL; visual mesh filename=package://rohand_urdf_ros2/meshes_l//mf_slider_link.STL
- link rf_connecting_link: geometry collision mesh filename=package://rohand_urdf_ros2/meshes_l//rf_connecting_link.STL; visual mesh filename=package://rohand_urdf_ros2/meshes_l//rf_connecting_link.STL
- link rf_distal_link: mass 0.00416255068209514 -> 0.00416255068346841; geometry collision mesh filename=package://rohand_urdf_ros2/meshes_l//rf_distal_link.STL; visual mesh filename=package://rohand_urdf_ros2/meshes_l//rf_distal_link.STL
- link rf_proximal_link: geometry collision mesh filename=package://rohand_urdf_ros2/meshes_l//rf_proximal_link.STL; visual mesh filename=package://rohand_urdf_ros2/meshes_l//rf_proximal_link.STL
- link rf_slider_abpart_link: geometry collision mesh filename=package://rohand_urdf_ros2/meshes_l//rf_slider_abpart_link.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; visual mesh filename=package://rohand_urdf_ros2/meshes_l//rf_slider_abpart_link.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
- link rf_slider_link: geometry collision mesh filename=package://rohand_urdf_ros2/meshes_l//rf_slider_link.STL; visual mesh filename=package://rohand_urdf_ros2/meshes_l//rf_slider_link.STL
- link th_connecting_link: geometry collision mesh filename=package://rohand_urdf_ros2/meshes_l//th_connecting_link.STL; visual mesh filename=package://rohand_urdf_ros2/meshes_l//th_connecting_link.STL
- link th_distal_link: mass 0.00503402600969819 -> 0.00503402601517063; geometry collision mesh filename=package://rohand_urdf_ros2/meshes_l//th_distal_link.STL; visual mesh filename=package://rohand_urdf_ros2/meshes_l//th_distal_link.STL
- link th_proximal_link: mass 0.00666243139311085 -> 0.00666243139310216; geometry collision mesh filename=package://rohand_urdf_ros2/meshes_l//th_proximal_link.STL; visual mesh filename=package://rohand_urdf_ros2/meshes_l//th_proximal_link.STL
- link th_root_link: mass 0.00231714462462064 -> 0.0021989478617719; geometry collision mesh filename=package://rohand_urdf_ros2/meshes_l//th_root_link.STL; visual mesh filename=package://rohand_urdf_ros2/meshes_l//th_root_link.STL
- link th_slider_link: geometry collision mesh filename=package://rohand_urdf_ros2/meshes_l//th_slider_link.STL; visual mesh filename=package://rohand_urdf_ros2/meshes_l//th_slider_link.STL
Joints:
- joint if_connecting_link: origin xyz=-0.120054040836567 0.0316923619468652 0.00321710545239118 rpy=-0.0872898030131476 -0.00722733820087602 -0.0823989405972364 -> xyz=-0.120051727129588 0.0318672321540881 0.00686116990260903 rpy=-0.0872898030131476 -0.00722733820087602 -0.0823989405972364
- joint if_proximal_link: origin xyz=-0.11269 0.030668 -0.0011639 rpy=-0.087311 -0.0072291 -0.082399 -> xyz=-0.112691326549452 0.0308429886174686 0.00248020890615535 rpy=-0.0873108596933026 -0.00722906372465864 -0.0823986361856106
- joint if_slider_link: origin xyz=-0.0931439129073844 0.0282184632206006 -0.00972507714068695 rpy=0 0 -0.0829795346970403 -> xyz=-0.093141599200405 0.0283933334278235 -0.0060810126904691 rpy=0 0 -0.0829795346970403
- joint lf_connecting_link: origin xyz=-0.1168 -0.030892 0.0042156 rpy=0.087244 -0.01033 0.11755 -> xyz=-0.11679 -0.030717 0.0078597 rpy=0.087244 -0.01033 0.11755
- joint lf_proximal_link: origin xyz=-0.10947 -0.029635 -0.00016701 rpy=0.087223 -0.010327 0.11755 -> xyz=-0.10947 -0.02946 0.0034771 rpy=0.087223 -0.010327 0.11755
- joint lf_slider_abpart_link: origin xyz=-0.0071723 0 0 rpy=0.087286 -0.010238 -0.00089593 -> xyz=-0.00717233182992167 0 0 rpy=0.087286192987255 -0.0102383843018635 -0.000895930220605248
- joint lf_slider_link: origin xyz=-0.089579 -0.026406 -0.0087232 rpy=0 -8.2704E-05 0.11831 -> xyz=-0.089576643926692 -0.0262308897592081 -0.00507914898073518 rpy=0 -8.27044529585942E-05 0.118308341349328
- joint mf_connecting_link: origin xyz=-0.12339 0.010594 0.0075442 rpy=2.1055E-05 0 -0.013245 -> xyz=-0.12339 0.010769 0.011188 rpy=2.1055E-05 0 -0.013245
- joint mf_proximal_link: origin xyz=-0.11597 0.010472 0.0031442 rpy=0 0 -0.013245 -> xyz=-0.11597 0.010647 0.0067882 rpy=0 0 -0.013245
- joint mf_slider_link: origin xyz=-0.095792 0.010329 -0.0054591 rpy=0 -0.00010039 -0.01323 -> xyz=-0.095789 0.010504 -0.001815 rpy=0 -0.00010039 -0.01323
- joint rf_connecting_link: origin xyz=-0.12065 -0.0097621 0.0067935 rpy=2.1021E-05 0 0.056602 -> xyz=-0.120646556392296 -0.00958718365665331 0.0104375725753832 rpy=2.10205544385047E-05 0 0.0566022572146075
- joint rf_proximal_link: origin xyz=-0.113238824661392 -0.00936892798564519 0.00239418207562177 rpy=0 0 0.056602255215157 -> xyz=-0.113236510954413 -0.00919405777842235 0.00603824652583962 rpy=0 0 0.056602255215157
- joint rf_slider_abpart_link: origin xyz=-0.0071723 0 0 rpy=-6.3003E-05 9.8956E-05 0 -> xyz=-0.00717233182914902 0 0 rpy=-6.30032465600259E-05 9.89558911798051E-05 0
- joint rf_slider_link: origin xyz=-0.093268 -0.0083093 -0.0062039 rpy=0 -9.5082E-05 0.056587 -> xyz=-0.093265347397978 -0.00813438556869404 -0.00255981174590743 rpy=0 -9.50818117190785E-05 0.0565869121559373
- joint th_connecting_link: origin xyz=0.0303 0.00016046 -0.000143 rpy=3.1387 -0.001435 2.6778 -> xyz=0.030299999929101 0.000160459585977893 -0.000142999395914452 rpy=3.13872334945882 -0.00143499623046761 2.67784667779356
- joint th_proximal_link: origin xyz=-0.0067545 0.02098 -0.0027 rpy=0 0 0.012931 -> xyz=-0.00675449620598668 0.0209804780594721 -0.00270002056556843 rpy=0 0 0.0129306539254238
- joint th_root_link: origin xyz=-0.046082 0.019841 -0.026844 rpy=0 -0.21841 -0.013245 -> xyz=-0.0460801443059001 0.020015956388997 -0.023200337031876 rpy=0 -0.218406428574065 -0.0132452733633124
- joint th_slider_link: origin xyz=-0.010802 0.0076387 -0.00016532 rpy=3.1384 0 2.6778 -> xyz=-0.0108023937111218 0.00763873324235342 -0.000165316557534618 rpy=3.13838452099804 0 2.67784461906022

File: urdf/rohand_right.urdf (robot description, URDF)
Before this commit: robot rohand_right, 26 links, 25 joints
Links:
- link base_link: mass 0.0365946767797895 -> 0.0365946767797888
- link if_connecting_link: mass 0.000247117851989123 -> 0.00024712
- link if_distal_link: mass 0.004164022259791 -> 0.00416402211038926
- link if_proximal_link: mass 0.00155087052217802 -> 0.0015509
- link if_slider_link: mass 0.0001919874302551 -> 0.00019199
- link lf_connecting_link: mass 0.000221221175136363 -> 0.00022122
- link lf_proximal_link: mass 0.00136675205423018 -> 0.0013668
- link lf_slider_link: mass 0.000191987419584901 -> 0.00019199
- link mf_connecting_link: mass 0.000270239292283242 -> 0.00027024
- link mf_distal_link: mass 0.00416397513493032 -> 0.00416397498628892
- link mf_proximal_link: mass 0.00189595262592985 -> 0.001896
- link mf_slider_link: mass 0.000191987434205271 -> 0.00019199
- link rf_connecting_link: mass 0.000247117839790627 -> 0.00024712
- link rf_distal_link: mass 0.00416283954000268 -> 0.00416283954044361
- link rf_proximal_link: mass 0.00155087002589292 -> 0.0015509
- link rf_slider_link: mass 0.000191987414464228 -> 0.00019199
- link th_distal_link: mass 0.00503423119409679 -> 0.00503423118877467
- link th_proximal_link: mass 0.00415628386649693 -> 0.0041563
- link th_root_link: mass 0.00231714411309494 -> 0.0021989
Joints:
- joint if_connecting_link: origin xyz=-0.12005 -0.031689 0.0031909 rpy=0.08729 -0.0072273 0.082399 -> xyz=-0.12005 -0.031698 0.0071031 rpy=0.08729 -0.0072273 0.082399
- joint if_proximal_link: origin xyz=-0.11269 -0.030664 -0.0011901 rpy=0.087311 -0.0072291 0.082399 -> xyz=-0.11269 -0.030673 0.0027221 rpy=0.087311 -0.0072291 0.082399
- joint if_slider_link: origin xyz=-0.093144 -0.028215 -0.0097513 rpy=0 0 0.08298 -> xyz=-0.093144 -0.028224 -0.0058391 rpy=0 0 0.08298
- joint lf_connecting_link: origin xyz=-0.1168 0.030896 0.0041893 rpy=-0.087244 -0.01033 -0.11755 -> xyz=-0.1168 0.030887 0.0081016 rpy=-0.087244 -0.01033 -0.11755
- joint lf_proximal_link: origin xyz=-0.10947 0.029638 -0.00019325 rpy=-0.087223 -0.010327 -0.11755 -> xyz=-0.10947 0.029629 0.003719 rpy=-0.087223 -0.010327 -0.11755
- joint lf_slider_link: origin xyz=-0.089579 0.026409 -0.0087495 rpy=0 -8.2704E-05 -0.11831 -> xyz=-0.089579 0.0264 -0.0048372 rpy=0 -8.2704E-05 -0.11831
- joint mf_connecting_link: origin xyz=-0.12339 -0.01059 0.007518 rpy=-2.1055E-05 0 0.013245 -> xyz=-0.12339 -0.010599 0.01143 rpy=-2.1055E-05 0 0.013245
- joint mf_proximal_link: origin xyz=-0.11597 -0.010469 0.0031179 rpy=0 0 0.013245 -> xyz=-0.11597 -0.010478 0.0070301 rpy=0 0 0.013245
- joint mf_slider_link: origin xyz=-0.095792 -0.010325 -0.0054853 rpy=0 -0.00010039 0.01323 -> xyz=-0.095792 -0.010334 -0.0015731 rpy=0 -0.00010039 0.01323
- joint rf_connecting_link: origin xyz=-0.12065 0.0097657 0.0067673 rpy=-2.1021E-05 0 -0.056602 -> xyz=-0.12065 0.0097568 0.010679 rpy=-2.1021E-05 0 -0.056602
- joint rf_proximal_link: origin xyz=-0.11324 0.0093726 0.0023679 rpy=0 0 -0.056602 -> xyz=-0.11324 0.0093636 0.0062802 rpy=0 0 -0.056602
- joint rf_slider_link: origin xyz=-0.093268 0.0083129 -0.0062301 rpy=0 -9.5082E-05 -0.056587 -> xyz=-0.093268 0.008304 -0.0023179 rpy=0 -9.5082E-05 -0.056587
- joint th_root_link: origin xyz=-0.046083 -0.019837 -0.026871 rpy=-0.0028701 -0.21841 0.013245 -> xyz=-0.046082 -0.019846 -0.022958 rpy=-0.0028701 -0.21841 0.013245

Commit message: Modified wrong joint angle limit.

File: urdf/rohand_left.urdf (robot description, URDF)
Before this commit: robot rohand_left, 26 links, 25 joints
Links:
- link base_link: mass 0.0518221802910333 -> 0.05182218018482; geometry collision mesh filename=package://rohand_urdf_ros2/meshes_l/base_link.STL; visual mesh filename=package://rohand_urdf_ros2/meshes_l/base_link.STL
- link if_connecting_link: geometry collision mesh filename=package://rohand_urdf_ros2/meshes_l/if_connecting_link.STL; visual mesh filename=package://rohand_urdf_ros2/meshes_l/if_connecting_link.STL
- link if_distal_link: mass 0.00416343809392657 -> 0.00416343809021936; geometry collision mesh filename=package://rohand_urdf_ros2/meshes_l/if_distal_link.STL; visual mesh filename=package://rohand_urdf_ros2/meshes_l/if_distal_link.STL
- link if_proximal_link: geometry collision mesh filename=package://rohand_urdf_ros2/meshes_l/if_proximal_link.STL; visual mesh filename=package://rohand_urdf_ros2/meshes_l/if_proximal_link.STL
- link if_slider_abpart_link: geometry collision mesh filename=package://rohand_urdf_ros2/meshes_l/if_slider_abpart_link.S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; visual mesh filename=package://rohand_urdf_ros2/meshes_l/if_slider_abpart_link.S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
- link if_slider_link: geometry collision mesh filename=package://rohand_urdf_ros2/meshes_l/if_slider_link.STL; visual mesh filename=package://rohand_urdf_ros2/meshes_l/if_slider_link.STL
- link lf_connecting_link: geometry collision mesh filename=package://rohand_urdf_ros2/meshes_l/lf_connecting_link.STL; visual mesh filename=package://rohand_urdf_ros2/meshes_l/lf_connecting_link.STL
- link lf_distal_link: geometry collision mesh filename=package://rohand_urdf_ros2/meshes_l/lf_distal_link.STL; visual mesh filename=package://rohand_urdf_ros2/meshes_l/lf_distal_link.STL
- link lf_proximal_link: geometry collision mesh filename=package://rohand_urdf_ros2/meshes_l/lf_proximal_link.STL; visual mesh filename=package://rohand_urdf_ros2/meshes_l/lf_proximal_link.STL
- link lf_slider_abpart_link: geometry collision mesh filename=package://rohand_urdf_ros2/meshes_l/lf_slider_abpart_link.S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; visual mesh filename=package://rohand_urdf_ros2/meshes_l/lf_slider_abpart_link.S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
- link lf_slider_link: geometry collision mesh filename=package://rohand_urdf_ros2/meshes_l/lf_slider_link.STL; visual mesh filename=package://rohand_urdf_ros2/meshes_l/lf_slider_link.STL
- link mf_connecting_link: geometry collision mesh filename=package://rohand_urdf_ros2/meshes_l/mf_connecting_link.STL; visual mesh filename=package://rohand_urdf_ros2/meshes_l/mf_connecting_link.STL
- link mf_distal_link: mass 0.0041634139178577 -> 0.00416341391410531; geometry collision mesh filename=package://rohand_urdf_ros2/meshes_l/mf_distal_link.STL; visual mesh filename=package://rohand_urdf_ros2/meshes_l/mf_distal_link.STL
- link mf_proximal_link: mass 0.102110343610594 -> 0.102110343400807; geometry collision mesh filename=package://rohand_urdf_ros2/meshes_l/mf_proximal_link.STL; visual mesh filename=package://rohand_urdf_ros2/meshes_l/mf_proximal_link.STL
- link mf_slider_abpart_link: geometry collision mesh filename=package://rohand_urdf_ros2/meshes_l/mf_slider_abpart_link.S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; visual mesh filename=package://rohand_urdf_ros2/meshes_l/mf_slider_abpart_link.S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
- link mf_slider_link: geometry collision mesh filename=package://rohand_urdf_ros2/meshes_l/mf_slider_link.STL; visual mesh filename=package://rohand_urdf_ros2/meshes_l/mf_slider_link.STL
- link rf_connecting_link: geometry collision mesh filename=package://rohand_urdf_ros2/meshes_l/rf_connecting_link.STL; visual mesh filename=package://rohand_urdf_ros2/meshes_l/rf_connecting_link.STL
- link rf_distal_link: mass 0.00416255068346841 -> 0.00416255068209514; geometry collision mesh filename=package://rohand_urdf_ros2/meshes_l/rf_distal_link.STL; visual mesh filename=package://rohand_urdf_ros2/meshes_l/rf_distal_link.STL
- link rf_proximal_link: geometry collision mesh filename=package://rohand_urdf_ros2/meshes_l/rf_proximal_link.STL; visual mesh filename=package://rohand_urdf_ros2/meshes_l/rf_proximal_link.STL
- link rf_slider_abpart_link: geometry collision mesh filename=package://rohand_urdf_ros2/meshes_l/rf_slider_abpart_link.S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; visual mesh filename=package://rohand_urdf_ros2/meshes_l/rf_slider_abpart_link.S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
- link rf_slider_link: geometry collision mesh filename=package://rohand_urdf_ros2/meshes_l/rf_slider_link.STL; visual mesh filename=package://rohand_urdf_ros2/meshes_l/rf_slider_link.STL
- link th_connecting_link: geometry collision mesh filename=package://rohand_urdf_ros2/meshes_l/th_connecting_link.STL; visual mesh filename=package://rohand_urdf_ros2/meshes_l/th_connecting_link.STL
- link th_distal_link: mass 0.00503402601517063 -> 0.00503402600969819; geometry collision mesh filename=package://rohand_urdf_ros2/meshes_l/th_distal_link.STL; visual mesh filename=package://rohand_urdf_ros2/meshes_l/th_distal_link.STL
- link th_proximal_link: mass 0.00666243139310216 -> 0.00666243139311084; geometry collision mesh filename=package://rohand_urdf_ros2/meshes_l/th_proximal_link.STL; visual mesh filename=package://rohand_urdf_ros2/meshes_l/th_proximal_link.STL
- link th_root_link: geometry collision mesh filename=package://rohand_urdf_ros2/meshes_l/th_root_link.STL; visual mesh filename=package://rohand_urdf_ros2/meshes_l/th_root_link.STL
- link th_slider_link: geometry collision mesh filename=package://rohand_urdf_ros2/meshes_l/th_slider_link.STL; visual mesh filename=package://rohand_urdf_ros2/meshes_l/th_slider_link.STL
Joints:
- joint if_connecting_link: origin xyz=-0.120051727129588 0.0318672321540881 0.00686116990260903 rpy=-0.0872898030131476 -0.00722733820087602 -0.0823989405972364 -> xyz=-0.12005 0.031867 0.0068612 rpy=-0.08729 -0.0072273 -0.082399
- joint if_distal_link: origin xyz=-0.0340605619485064 0 -0.0114050053411428 rpy=2.57804029017016E-05 0 -0.000101940406116998 -> xyz=-0.034061 0 -0.011405 rpy=2.578E-05 0 -0.00010194
- joint if_proximal_link: origin xyz=-0.112691326549452 0.0308429886174686 0.00248020890615535 rpy=-0.0873108596933026 -0.00722906372465864 -0.0823986361856106 -> xyz=-0.11269 0.030843 0.0024802 rpy=-0.087311 -0.0072291 -0.082399
- joint if_slider_abpart_link: origin xyz=-0.00717233182793718 0 0 rpy=-0.0872362806506897 -0.00722294993772634 0.000631700989182225 -> xyz=-0.0071723 0 0 rpy=-0.087236 -0.0072229 0.0006317
- joint if_slider_link: origin xyz=-0.093141599200405 0.0283933334278235 -0.0060810126904691 rpy=0 0 -0.0829795346970403 -> xyz=-0.093142 0.028393 -0.006081 rpy=0 0 -0.08298
- joint lf_slider_abpart_link: origin xyz=-0.00717233182992167 0 0 rpy=0.087286192987255 -0.0102383843018635 -0.000895930220605248 -> xyz=-0.0071723 0 0 rpy=0.087286 -0.010238 -0.00089593
- joint lf_slider_link: origin xyz=-0.089576643926692 -0.0262308897592081 -0.00507914898073518 rpy=0 -8.27044529585942E-05 0.118308341349328 -> xyz=-0.089577 -0.026231 -0.0050791 rpy=0 -8.2704E-05 0.11831
- joint rf_connecting_link: origin xyz=-0.120646556392296 -0.00958718365665331 0.0104375725753832 rpy=2.10205544385047E-05 0 0.0566022572146075 -> xyz=-0.12065 -0.0095872 0.010438 rpy=2.1021E-05 0 0.056602
- joint rf_distal_link: origin xyz=-0.0336433389681109 0 -0.0125825979097555 rpy=2.93098936036424E-05 0 -0.0001009823092024 -> xyz=-0.033643 0 -0.012583 rpy=2.931E-05 0 -0.00010098
- joint rf_proximal_link: origin xyz=-0.113236510954413 -0.00919405777842235 0.00603824652583962 rpy=0 0 0.056602255215157 -> xyz=-0.11324 -0.0091941 0.0060382 rpy=0 0 0.056602
- joint rf_slider_abpart_link: origin xyz=-0.00717233182914902 0 0 rpy=-6.30032465600259E-05 9.89558911798051E-05 0 -> xyz=-0.0071723 0 0 rpy=-6.3003E-05 9.8956E-05 0
- joint rf_slider_link: origin xyz=-0.093265347397978 -0.00813438556869404 -0.00255981174590743 rpy=0 -9.50818117190785E-05 0.0565869121559373 -> xyz=-0.093265 -0.0081344 -0.0025598 rpy=0 -9.5082E-05 0.056587
- joint th_connecting_link: origin xyz=0.030299999929101 0.000160459585977893 -0.000142999395914452 rpy=3.13872334945882 -0.00143499623046761 2.67784667779356 -> xyz=0.0303 0.00016046 -0.000143 rpy=3.1387 -0.001435 2.6778
- joint th_proximal_link: origin xyz=-0.00675449620598668 0.0209804780594721 -0.00270002056556843 rpy=0 0 0.0129306539254238 -> xyz=-0.0067545 0.02098 -0.0027 rpy=0 0 0.012931
- joint th_root_link: origin xyz=-0.0460801443059001 0.020015956388997 -0.023200337031876 rpy=0 -0.218406428574065 -0.0132452733633124 -> xyz=-0.04608 0.020016 -0.0232 rpy=0 -0.21841 -0.013245
- joint th_slider_link: origin xyz=-0.0108023937111218 0.00763873324235342 -0.000165316557534618 rpy=3.13838452099804 0 2.67784461906022 -> xyz=-0.010802 0.0076387 -0.00016532 rpy=3.1384 0 2.6778

File: urdf/rohand_right.urdf (robot description, URDF)
Before this commit: robot rohand_right, 26 links, 25 joints
Links:
- link base_link: mass 0.0365946767797888 -> 0.036595
- link if_connecting_link: mass 0.00024712 -> 0.000247117851989122
- link if_proximal_link: mass 0.0015509 -> 0.00155087052217806
- link lf_connecting_link: mass 0.00022122 -> 0.000221221175136363
- link lf_proximal_link: mass 0.0013668 -> 0.00136675205423018
- link lf_slider_link: mass 0.00019199 -> 0.000191987419584901
- link mf_connecting_link: mass 0.00027024 -> 0.000270239292283242
- link mf_proximal_link: mass 0.001896 -> 0.00189595262592985
- link mf_slider_link: mass 0.00019199 -> 0.000191987434205271
- link rf_connecting_link: mass 0.00024712 -> 0.000247117839790627
- link rf_distal_link: mass 0.00416283954044361 -> 0.0041628395404436
- link rf_proximal_link: mass 0.0015509 -> 0.00155087002589296
- link rf_slider_link: mass 0.00019199 -> 0.000191987414464228
- link th_proximal_link: mass 0.0041563 -> 0.00415628386649693
- link th_root_link: mass 0.0021989 -> 0.0021989473502463
Joints:
- joint if_distal_link: limit lower=-1.57 upper=1.57 effort=0 velocity=0 -> lower=0 upper=0 effort=0 velocity=0
- joint if_proximal_link: limit lower=-1.57 upper=1.57 effort=0 velocity=0 -> lower=0 upper=0 effort=0 velocity=0
- joint if_slider_abpart_link: limit lower=-1.57 upper=1.57 effort=0 velocity=0 -> lower=0 upper=0 effort=0 velocity=0
