Commit message: Adjust the initial posture to open

File: urdf/rohand_left.urdf (robot description, URDF)
Before this commit: robot rohand_left, 26 links, 25 joints
Links:
- link base_link: mass 0.05182218018482 -> 0.0559618850522869
- link if_connecting_link: mass 0.00024711756965943 -> 0.000197692348310411
- link if_distal_link: mass 0.00416343809021936 -> 0.0042269383122795
- link if_proximal_link: mass 0.00155055071205295 -> 0.00154987032874225
- link if_slider_abpart_link: mass 0.000457378818734687 -> 0.000419595822746572
- link if_slider_link: mass 0.000191988555317022 -> 0.00048911221771827
- link lf_connecting_link: mass 0.000221227665967327 -> 0.000176980932045691
- link lf_distal_link: mass 0.00263003416842098 -> 0.00262042947413116
- link lf_proximal_link: mass 0.00136673401761359 -> 0.00136661208486985
- link lf_slider_abpart_link: mass 0.000457378802064142 -> 0.000419595826532552
- link lf_slider_link: mass 0.000191988562577953 -> 0.000510662528391611
- link mf_connecting_link: mass 0.000270250689971117 -> 0.000216184518525667
- link mf_distal_link: mass 0.00416341391410531 -> 0.0042269628029676
- link mf_proximal_link: mass 0.102110343400807 -> 0.00189508780970619
- link mf_slider_abpart_link: mass 0.000457378814740125 -> 0.000419595848489683
- link mf_slider_link: mass 0.000191988548040141 -> 0.000489112305392741
- link rf_connecting_link: mass 0.000247117666203693 -> 0.000197692354337264
- link rf_distal_link: mass 0.00416255068209514 -> 0.00422730983553646
- link rf_proximal_link: mass 0.00155057954584347 -> 0.00154985371268108
- link rf_slider_abpart_link: mass 0.000457378802308313 -> 0.000419595841745906
- link rf_slider_link: mass 0.000191988559777486 -> 0.000489112303078988
- link th_connecting_link: mass 0.000339219041152736 -> 0.000334843777726033
- link th_distal_link: mass 0.00503402600969819 -> 0.00509494222453049
- link th_proximal_link: mass 0.00666243139311084 -> 0.00501318922026079
- link th_root_link: mass 0.0021989478617719 -> 0.00217782401907458
- link th_slider_link: mass 0.00106238517527826 -> 0.000966918573679237
Joints:
- joint if_connecting_link: axis 0 1 0 -> 0.082428 0.99278 -0.087177; origin xyz=-0.12005 0.031867 0.0068612 rpy=-0.08729 -0.0072273 -0.082399 -> xyz=-0.11976 0.03521 0.0028896 rpy=0 0 0
- joint if_distal_link: axis 0 1 0 -> 0.082428 0.99278 -0.087177; origin xyz=-0.034061 0 -0.011405 rpy=2.578E-05 0 -0.00010194 -> xyz=-0.035776 0.0028401 -0.0014841 rpy=0 0 0
- joint if_proximal_link: axis 0 1 0 -> 0.082428 0.99278 -0.087177; origin xyz=-0.11269 0.030843 0.0024802 rpy=-0.087311 -0.0072291 -0.082399 -> xyz=-0.11211 0.037738 -0.0018032 rpy=0 0 0
- joint if_slider_abpart_link: axis 0 1 0 -> 0.082734 0.99276 -0.087135; origin xyz=-0.0071723 0 0 rpy=-0.087236 -0.0072229 0.0006317 -> xyz=-0.02861 0.0058839 -0.00030477 rpy=0 0 0
- joint if_slider_link: axis 1 0 0 -> 0.99655 -0.083049 0; limit lower=-0.003 upper=0.016 effort=0 velocity=0 -> lower=0 upper=0.019 effort=0 velocity=0; origin xyz=-0.093142 0.028393 -0.006081 rpy=0 0 -0.08298 -> xyz=-0.074396 0.026655 -0.0097434 rpy=0 0 0
- joint lf_connecting_link: axis 0 1 0 -> -0.11759 0.98924 0.087085; origin xyz=-0.11679 -0.030717 0.0078597 rpy=0.087244 -0.01033 0.11755 -> xyz=-0.11723 -0.027174 0.0045247 rpy=0 0 0
- joint lf_distal_link: axis 0 1 0 -> -0.11759 0.98923 0.087106; origin xyz=-0.029737 5.0315E-05 -0.011632 rpy=2.1055E-05 0 0 -> xyz=-0.031562 -0.0034532 -0.003392 rpy=0 0 0
- joint lf_proximal_link: axis 0 1 0 -> -0.11759 0.98923 0.087106; origin xyz=-0.10947 -0.02946 0.0034771 rpy=0.087223 -0.010327 0.11755 -> xyz=-0.11032 -0.022406 0.00045133 rpy=0 0 0
- joint lf_slider_abpart_link: axis 0 1 0 -> -0.11759 0.98923 0.08715; origin xyz=-0.0071723 0 0 rpy=0.087286 -0.010238 -0.00089593 -> xyz=-0.029209 4.0116E-05 0.00030326 rpy=0 0 0
- joint lf_slider_link: axis 1 0 0 -> 0.99301 0.11803 8.2704E-05; limit lower=-0.003 upper=0.016 effort=0 velocity=0 -> lower=0 upper=0.019 effort=0 velocity=0; origin xyz=-0.089577 -0.026231 -0.0050791 rpy=0 -8.2704E-05 0.11831 -> xyz=-0.070847 -0.024182 -0.0087399 rpy=0 0 0
- joint mf_connecting_link: axis 0 1 0 -> 0.013244 0.99991 2.1054E-05; origin xyz=-0.12339 0.010769 0.011188 rpy=2.1055E-05 0 -0.013245 -> xyz=-0.12334 0.014341 0.0075259 rpy=0 0 0
- joint mf_distal_link: axis 0 1 0 -> 0.013244 0.99991 2.1055E-05; origin xyz=-0.038293 0 -0.014673 rpy=0 0 0 -> xyz=-0.040851 0.00054126 -0.0035367 rpy=0 0 0
- joint mf_proximal_link: axis 0 1 0 -> 0.013244 0.99991 4.2699E-05; origin xyz=-0.11597 0.010647 0.0067882 rpy=0 0 -0.013245 -> xyz=-0.11587 0.017792 0.0031262 rpy=0 0 0
- joint mf_slider_abpart_link: axis 0 1 0 -> 0.013228 0.99991 -7.2594E-05; origin xyz=-0.0071723 0 0 rpy=-6.2891E-05 9.9576E-05 0 -> xyz=-0.028951 0.0038841 0 rpy=0 0 0
- joint mf_slider_link: axis 1 0 0 -> 0.99991 -0.013228 0.00010039; limit lower=-0.003 upper=0.016 effort=0 velocity=0 -> lower=0 upper=0.019 effort=0 velocity=0; origin xyz=-0.095789 0.010504 -0.001815 rpy=0 -0.00010039 -0.01323 -> xyz=-0.076974 0.010077 -0.0054756 rpy=0 0 0
- joint rf_connecting_link: axis 0 1 0 -> -0.05658 0.9984 2.102E-05; origin xyz=-0.12065 -0.0095872 0.010438 rpy=2.1021E-05 0 0.056602 -> xyz=-0.11723 -0.027174 0.0045247 rpy=0 0 0
- joint rf_distal_link: axis 0 1 0 -> -0.05658 0.9984 2.102E-05; origin xyz=-0.033643 0 -0.012583 rpy=2.931E-05 0 -0.00010098 -> xyz=-0.035766 -0.0020268 -0.0026198 rpy=0 0 0
- joint rf_proximal_link: axis 0 1 0 -> -0.05658 0.9984 2.102E-05; origin xyz=-0.11324 -0.0091941 0.0060382 rpy=0 0 0.056602 -> xyz=-0.11364 -0.0022565 0.0023761 rpy=0 0 0
- joint rf_slider_abpart_link: axis 0 1 0 -> -0.056554 0.9984 -7.942E-05; origin xyz=-0.0071723 0 0 rpy=-6.3003E-05 9.8956E-05 0 -> xyz=-0.029152 0.0018551 0 rpy=0 0 0
- joint rf_slider_link: axis 1 0 0 -> 0.9984 0.056554 9.5082E-05; limit lower=-0.003 upper=0.016 effort=0 velocity=0 -> lower=0 upper=0.019 effort=0 velocity=0; origin xyz=-0.093265 -0.0081344 -0.0025598 rpy=0 -9.5082E-05 0.056587 -> xyz=-0.074498 -0.0072492 -0.0062204 rpy=0 0 0
- joint th_connecting_link: axis 0 0 -1 -> 0.21699 0.032029 -0.97565; origin xyz=0.0303 0.00016046 -0.000143 rpy=3.1387 -0.001435 2.6778 -> xyz=-0.027697 0.024088 -0.010084 rpy=0 0 0
- joint th_distal_link: axis 0 0 -1 -> 0.21698 0.032029 -0.97565; origin xyz=-0.050881 0.013011 -0.0020153 rpy=0 0 0 -> xyz=-0.00010351 0.023735 -0.046849 rpy=0 -1.352 -0.032034
- joint th_proximal_link: axis 0 0 -1 -> 1 0 0; origin xyz=-0.0067545 0.02098 -0.0027 rpy=0 0 0.012931 -> xyz=-0.025097 0.021667 -0.015581 rpy=0.14303 1.3497 0.14655
- joint th_root_link: axis -1 0 0 -> -0.97616 0.01293 -0.21667; limit lower=-0.035 upper=1.605 effort=0 velocity=0 -> lower=0 upper=1.57 effort=0 velocity=0; origin xyz=-0.04608 0.020016 -0.0232 rpy=0 -0.21841 -0.013245 -> xyz=-0.024656 0.019554 -0.022107 rpy=0 0 0
- joint th_slider_link: axis 1 0 0 -> -0.761977793105663 0.630282689066857 -0.148773568473957; limit lower=-0.003 upper=0.008 effort=0 velocity=0 -> lower=0 upper=0.01 effort=0 velocity=0; origin xyz=-0.010802 0.0076387 -0.00016532 rpy=3.1384 0 2.6778 -> xyz=-0.0076999999999972 0.00276927591433551 -0.000236666241639902 rpy=0 -1.3519569747769 -0.0320343601595158

File: urdf/rohand_right.urdf (robot description, URDF)
Before this commit: robot rohand_right, 26 links, 25 joints
Links:
- link base_link: mass 0.036595 -> 0.0941614898718946
- link if_connecting_link: mass 0.000247117851989122 -> 0.000197689248381643
- link if_distal_link: mass 0.00416402211038926 -> 0.00486631616894411
- link if_proximal_link: mass 0.00155087052217806 -> 0.00154952958352476
- link if_slider_abpart_link: mass 0.000457378804599453 -> 0.000526636346253179
- link if_slider_link: mass 0.00019199 -> 0.000489138281878773
- link lf_connecting_link: mass 0.000221221175136363 -> 0.000176981602686642
- link lf_distal_link: mass 0.00263003860844415 -> 0.00326999621591245
- link lf_proximal_link: mass 0.00136675205423018 -> 0.00136677973237
- link lf_slider_abpart_link: mass 0.000457378787584006 -> 0.000526636335571007
- link lf_slider_link: mass 0.000191987419584901 -> 0.000489138222296884
- link mf_connecting_link: mass 0.000270239292283242 -> 0.000216186298115104
- link mf_distal_link: mass 0.00416397498628892 -> 0.00486610881870854
- link mf_proximal_link: mass 0.00189595262592985 -> 0.00189501857338832
- link mf_slider_abpart_link: mass 0.000457378800703002 -> 0.000526636368526203
- link mf_slider_link: mass 0.000191987434205271 -> 0.000489138286069735
- link rf_connecting_link: mass 0.000247117839790627 -> 0.000197689252304948
- link rf_distal_link: mass 0.0041628395404436 -> 0.00486607601001256
- link rf_proximal_link: mass 0.00155087002589296 -> 0.0015495346822944
- link rf_slider_abpart_link: mass 0.000457378787987907 -> 0.000526636350514617
- link rf_slider_link: mass 0.000191987414464228 -> 0.000489138255422532
- link th_connecting_link: mass 0.000339222396740572 -> 0.000607798102631607
- link th_distal_link: mass 0.00503423118877467 -> 0.00601772502419511
- link th_proximal_link: mass 0.00415628386649693 -> 0.00501307756145889
- link th_root_link: mass 0.0021989473502463 -> 0.00217782328356739
- link th_slider_link: mass 0.00106239517277624 -> 0.000966927715708797
Joints:
- joint if_connecting_link: axis 0 1 0 -> -0.082428 0.99278 0.087177; origin xyz=-0.12005 -0.031698 0.0071031 rpy=0.08729 -0.0072273 0.082399 -> xyz=-0.12029 -0.028806 0.0072922 rpy=0 0 0
- joint if_distal_link: axis 0 1 0 -> -0.082428 0.99278 0.087177; limit lower=0 upper=0 effort=0 velocity=0 -> (none); origin xyz=-0.034061 0 -0.011405 rpy=-2.578E-05 0 0.00010194 -> xyz=-0.035776 -0.0028401 -0.0014841 rpy=0 0 0
- joint if_proximal_link: axis 0 1 0 -> -0.082428 0.99278 0.087177; limit lower=0 upper=0 effort=0 velocity=0 -> (none); origin xyz=-0.11269 -0.030673 0.0027221 rpy=0.087311 -0.0072291 0.082399 -> xyz=-0.11324 -0.024137 0.0032314 rpy=0 0 0
- joint if_slider_abpart_link: axis 0 1 0 -> -0.082734 0.99276 0.087135; limit lower=0 upper=0 effort=0 velocity=0 -> (none); origin xyz=-0.0071723 0 0 rpy=0.087236 -0.0072229 -0.0006317 -> xyz=-0.029189 0.0010654 0.00030518 rpy=0 0 0
- joint if_slider_link: axis 1 0 0 -> 0.99655 0.083049 0; limit lower=-0.003 upper=0.016 effort=0 velocity=0 -> lower=0 upper=0.019 effort=0 velocity=0; origin xyz=-0.093144 -0.028224 -0.0058391 rpy=0 0 0.08298 -> xyz=-0.074396 -0.026655 -0.0059032 rpy=0 0 0
- joint lf_connecting_link: axis 0 1 0 -> 0.11759 0.98924 -0.087085; origin xyz=-0.1168 0.030887 0.0081016 rpy=-0.087244 -0.01033 -0.11755 -> xyz=-0.11647 0.033555 0.0078033 rpy=0 0 0
- joint lf_distal_link: axis 0 1 0 -> 0.11759 0.98923 -0.087106; origin xyz=-0.029737 -5.0315E-05 -0.011632 rpy=-2.1055E-05 0 0 -> xyz=-0.031562 0.0034532 -0.003392 rpy=0 0 0
- joint lf_proximal_link: axis 0 1 0 -> 0.117591058209323 0.989234457465869 -0.0871064359930968; origin xyz=-0.10947 0.029629 0.003719 rpy=-0.087223 -0.010327 -0.11755 -> xyz=-0.10871130258864 0.0359583660197833 0.00309824490260681 rpy=0 0 0
- joint lf_slider_abpart_link: axis 0 1 0 -> 0.117590610595967 0.989230669602698 -0.0871500465694956; origin xyz=-0.0071723 0 0 rpy=-0.087286 -0.010238 0.00089593 -> xyz=-0.0283858043783233 0.00688449840682251 -0.000306788289491815 rpy=0 0 0
- joint lf_slider_link: axis 1 0 0 -> 0.993009723934899 -0.118032543523823 8.27044911595336E-05; limit lower=-0.003 upper=0.016 effort=0 velocity=0 -> lower=0 upper=0.019 effort=0 velocity=0; origin xyz=-0.089579 0.0264 -0.0048372 rpy=0 -8.2704E-05 -0.11831 -> xyz=-0.0708466334619896 0.0241824111749996 -0.00489967270216645 rpy=0 0 0
- joint mf_connecting_link: axis 0 1 0 -> -0.013244 0.99991 -2.1054E-05; origin xyz=-0.12339 -0.010599 0.01143 rpy=-2.1055E-05 0 0.013245 -> xyz=-0.12342 -0.0078912 0.011366 rpy=0 0 0
- joint mf_distal_link: axis 0 1 0 -> -0.013244 0.99991 -2.1055E-05; origin xyz=-0.038293 0 -0.014673 rpy=0 0 0 -> xyz=-0.040851 -0.00054126 -0.0035364 rpy=0 0 0
- joint mf_proximal_link: axis 0 1 0 -> -0.013244 0.99991 -4.2699E-05; origin xyz=-0.11597 -0.010478 0.0070301 rpy=0 0 0.013245 -> xyz=-0.11605 -0.0040932 0.0069659 rpy=0 0 0
- joint mf_slider_abpart_link: axis 0 1 0 -> -0.013228 0.99991 7.2594E-05; origin xyz=-0.0071723 0 0 rpy=6.2891E-05 9.9576E-05 0 -> xyz=-0.029044 0.0031153 0 rpy=0 0 0
- joint mf_slider_link: axis 1 0 0 -> 0.99991 0.013228 0.00010039; limit lower=-0.003 upper=0.016 effort=0 velocity=0 -> lower=0 upper=0.019 effort=0 velocity=0; origin xyz=-0.095792 -0.010334 -0.0015731 rpy=0 -0.00010039 0.01323 -> xyz=-0.076974 -0.010077 -0.0016353 rpy=0 0 0
- joint rf_connecting_link: axis 0 1 0 -> 0.0565797489260885 0.99839808271532 -2.10198201110756E-05; origin xyz=-0.12065 0.0097568 0.010679 rpy=-2.1021E-05 0 -0.056602 -> xyz=-0.1204851022382 0.0126604995038233 0.0106153804877178 rpy=0 0 0
- joint rf_distal_link: axis 0 1 0 -> 0.05658 0.9984 -2.102E-05; origin xyz=-0.033643 0 -0.012583 rpy=-2.931E-05 0 0.00010098 -> xyz=-0.035766 0.0020268 -0.0026198 rpy=0 0 0
- joint rf_proximal_link: axis 0 1 0 -> 0.05658 0.9984 -2.102E-05; origin xyz=-0.11324 0.0093636 0.0062802 rpy=0 0 -0.056602 -> xyz=-0.11287 0.015935 0.0062161 rpy=0 0 0
- joint rf_slider_abpart_link: axis 0 1 0 -> 0.056554 0.9984 7.942E-05; origin xyz=-0.0071723 0 0 rpy=6.3003E-05 9.8956E-05 0 -> xyz=-0.028756 0.0051336 0 rpy=0 0 0
- joint rf_slider_link: axis 1 0 0 -> 0.9984 -0.056554 9.5082E-05; limit lower=-0.003 upper=0.016 effort=0 velocity=0 -> lower=0 upper=0.019 effort=0 velocity=0; origin xyz=-0.093268 0.008304 -0.0023179 rpy=0 -9.5082E-05 -0.056587 -> xyz=-0.074498 0.0072492 -0.0023801 rpy=0 0 0
- joint th_connecting_link: axis 0 0 -1 -> -0.21699 0.032029 0.97565; origin xyz=0.0303 0.00014544 0.00015825 rpy=-3.0553 0.043068 -0.46189 -> xyz=-0.026144 -0.020984 -0.0010258 rpy=0 0 0
- joint th_distal_link: axis 0 0 -1 -> -0.21698 0.032029 0.97565; origin xyz=0.050881 -0.013011 0.0020153 rpy=0 0 0 -> xyz=-0.049076 -0.023254 0.004868 rpy=0 0 0
- joint th_proximal_link: axis 0 0 -1 -> -0.21699 -0.032029 0.97565; origin xyz=-0.0067545 -0.020973 -0.0027602 rpy=3.1387 -3.7078E-05 3.1287 -> xyz=-0.025097 -0.021667 -0.015581 rpy=0 0 0
- joint th_root_link: axis 1 0 0 -> 0.97616 0.01293 0.21667; limit lower=-0.034 upper=1.605 effort=0 velocity=0 -> lower=0 upper=1.57 effort=0 velocity=0; origin xyz=-0.046082 -0.019846 -0.022958 rpy=-0.0028701 -0.21841 0.013245 -> xyz=-0.024656 -0.019554 -0.018266 rpy=0 0 0
- joint th_slider_link: axis 1 0 0 -> -0.76198 -0.63028 -0.14877; limit lower=-0.003 upper=0.008 effort=0 velocity=0 -> lower=0 upper=0.01 effort=0 velocity=0; origin xyz=0.010802 -0.0076387 0.00016532 rpy=3.0452 0 -0.46375 -> xyz=-0.0053401 -0.0053494 0.0068801 rpy=0 0 0
